File: heehaw10/heehaw10.brd (EAGLE design)
At the start: 35.6 x 17.8 mm, 19 parts, among them J1 JST-SH-4, J2 PHD_1X7, J3 PHD_1X7, U1 AP2112SOT25

Commit message: move stuff
Parts:
- C2, C3: value (none) -> 10uF
- R1, R2, R5: value (none) -> 10k
- R4: value (none) -> 1k
Changed lines of the file:
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@@
 </autorouter>
 <elements>
-<element name="C2" library="rcl" library_urn="urn:adsk.eagle:library:334" package="C0603" package3d_urn="urn:adsk.eagle:package:23616/2" value="" x="8.382" y="12.7" smashed="yes">
+<element name="C2" library="rcl" library_urn="urn:adsk.eagle:library:334" package="C0603" package3d_urn="urn:adsk.eagle:package:23616/2" value="10uF" x="8.382" y="12.7" smashed="yes">
 <attribute name="POPULARITY" value="73" x="23.622" y="-17.78" size="1.778" layer="27" display="off"/>
 <attribute name="SPICEPREFIX" value="C" x="23.622" y="-17.78" size="1.778" layer="27" display="off"/>
 <attribute name="VALUE" x="7.747" y="10.795" size="1.27" layer="27"/>
 </element>
-<element name="C3" library="rcl" library_urn="urn:adsk.eagle:library:334" package="C0603" package3d_urn="urn:adsk.eagle:package:23616/2" value="" x="13.97" y="3.81" smashed="yes" rot="R270">
+<element name="C3" library="rcl" library_urn="urn:adsk.eagle:library:334" package="C0603" package3d_urn="urn:adsk.eagle:package:23616/2" value="10uF" x="13.97" y="3.81" smashed="yes" rot="R270">
 <attribute name="POPULARITY" value="73" x="-16.51" y="-15.24" size="1.778" layer="27" rot="R270" display="off"/>
 <attribute name="SPICEPREFIX" value="C" x="-16.51" y="-15.24" size="1.778" layer="27" rot="R270" display="off"/>
@@
 <attribute name="VALUE" x="14.097" y="11.43" size="0.4064" layer="27" ratio="10"/>
 </element>
-<element name="R1" library="rcl" library_urn="urn:adsk.eagle:library:334" package="R0603" package3d_urn="urn:adsk.eagle:package:23555/3" value="" x="23.495" y="10.922" smashed="yes" rot="R180">
+<element name="R1" library="rcl" library_urn="urn:adsk.eagle:library:334" package="R0603" package3d_urn="urn:adsk.eagle:package:23555/3" value="10k" x="23.495" y="10.922" smashed="yes" rot="R180">
 <attribute name="POPULARITY" value="70" x="0.635" y="41.402" size="1.778" layer="27" rot="R180" display="off"/>
 <attribute name="SPICEPREFIX" value="R" x="0.635" y="41.402" size="1.778" layer="27" rot="R180" display="off"/>
 <attribute name="VALUE" x="24.13" y="12.827" size="1.27" layer="27" rot="R180"/>
 </element>
-<element name="R2" library="rcl" library_urn="urn:adsk.eagle:library:334" package="R0603" package3d_urn="urn:adsk.eagle:package:23555/3" value="" x="20.574" y="12.954" smashed="yes" rot="R180">
+<element name="R2" library="rcl" library_urn="urn:adsk.eagle:library:334" package="R0603" package3d_urn="urn:adsk.eagle:package:23555/3" value="10k" x="20.574" y="12.954" smashed="yes" rot="R180">
 <attribute name="POPULARITY" value="70" x="-6.096" y="43.434" size="1.778" layer="27" rot="R180" display="off"/>
 <attribute name="SPICEPREFIX" value="R" x="-6.096" y="43.434" size="1.778" layer="27" rot="R180" display="off"/>
@@
 <attribute name="VALUE" x="26.416" y="10.922" size="1.27" layer="27"/>
 </element>
-<element name="R4" library="rcl" library_urn="urn:adsk.eagle:library:334" package="R0603" package3d_urn="urn:adsk.eagle:package:23555/3" value="" x="7.62" y="5.969" smashed="yes" rot="R180">
+<element name="R4" library="rcl" library_urn="urn:adsk.eagle:library:334" package="R0603" package3d_urn="urn:adsk.eagle:package:23555/3" value="1k" x="7.62" y="5.969" smashed="yes" rot="R180">
 <attribute name="POPULARITY" value="70" x="-26.67" y="36.449" size="1.778" layer="27" rot="R180" display="off"/>
 <attribute name="SPICEPREFIX" value="R" x="-26.67" y="36.449" size="1.778" layer="27" rot="R180" display="off"/>
 <attribute name="VALUE" x="8.255" y="7.874" size="1.27" layer="27" rot="R180"/>
 </element>
-<element name="R5" library="Ooo-Resistors" package="RESPACK_4X0603" value="" x="12.446" y="8.128" smashed="yes" rot="R270">
+<element name="R5" library="Ooo-Resistors" package="RESPACK_4X0603" value="10k" x="12.446" y="8.128" smashed="yes" rot="R270">
 <attribute name="VALUE" x="10.046" y="9.728" size="0.8128" layer="27" font="vector" ratio="10" rot="R270"/>
 </element>
