File: heehaw10/heehaw10.sch (EAGLE design)
At the start: 19 parts, among them J1 JST-SH-4, J2 PHD_1X7, J3 PHD_1X7, U1 AP2112SOT25

Commit message: move stuff
Parts:
- C2, C3: value (none) -> 10uF
- R1, R2, R5: value (none) -> 10k
- R4: value (none) -> 1k
Changed lines of the file:
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@@
 <part name="X2" library="Ooo-Connectors" deviceset="SWD_2X5" device=""/>
 <part name="U$2" library="Ooo-Switches" deviceset="PTS647" device=""/>
-<part name="R1" library="rcl" library_urn="urn:adsk.eagle:library:334" deviceset="R-EU_" device="R0603" package3d_urn="urn:adsk.eagle:package:23555/3"/>
-<part name="C2" library="rcl" library_urn="urn:adsk.eagle:library:334" deviceset="C-EU" device="C0603" package3d_urn="urn:adsk.eagle:package:23616/2"/>
-<part name="C3" library="rcl" library_urn="urn:adsk.eagle:library:334" deviceset="C-EU" device="C0603" package3d_urn="urn:adsk.eagle:package:23616/2"/>
+<part name="R1" library="rcl" library_urn="urn:adsk.eagle:library:334" deviceset="R-EU_" device="R0603" package3d_urn="urn:adsk.eagle:package:23555/3" value="10k"/>
+<part name="C2" library="rcl" library_urn="urn:adsk.eagle:library:334" deviceset="C-EU" device="C0603" package3d_urn="urn:adsk.eagle:package:23616/2" value="10uF"/>
+<part name="C3" library="rcl" library_urn="urn:adsk.eagle:library:334" deviceset="C-EU" device="C0603" package3d_urn="urn:adsk.eagle:package:23616/2" value="10uF"/>
 <part name="U$5" library="Ooo-PowerSymbols" deviceset="3.3V" device=""/>
 <part name="U$7" library="Ooo-PowerSymbols" deviceset="GND" device=""/>
@@
 <part name="U$10" library="Ooo-PowerSymbols" deviceset="3.3V" device=""/>
 <part name="U$11" library="Ooo-PowerSymbols" deviceset="GND" device=""/>
-<part name="R2" library="rcl" library_urn="urn:adsk.eagle:library:334" deviceset="R-EU_" device="R0603" package3d_urn="urn:adsk.eagle:package:23555/3"/>
+<part name="R2" library="rcl" library_urn="urn:adsk.eagle:library:334" deviceset="R-EU_" device="R0603" package3d_urn="urn:adsk.eagle:package:23555/3" value="10k"/>
 <part name="U$12" library="Ooo-PowerSymbols" deviceset="3.3V" device=""/>
 <part name="U$15" library="Ooo-PowerSymbols" deviceset="GND" device=""/>
 <part name="R3" library="rcl" library_urn="urn:adsk.eagle:library:334" deviceset="R-EU_" device="R0603" package3d_urn="urn:adsk.eagle:package:23555/3"/>
-<part name="R4" library="rcl" library_urn="urn:adsk.eagle:library:334" deviceset="R-EU_" device="R0603" package3d_urn="urn:adsk.eagle:package:23555/3"/>
+<part name="R4" library="rcl" library_urn="urn:adsk.eagle:library:334" deviceset="R-EU_" device="R0603" package3d_urn="urn:adsk.eagle:package:23555/3" value="1k"/>
 <part name="U$16" library="Ooo-PowerSymbols" deviceset="3.3V" device=""/>
 <part name="U$17" library="Ooo-PowerSymbols" deviceset="GND" device=""/>
@@
 <part name="U$14" library="Ooo-PowerSymbols" deviceset="GND" device=""/>
 <part name="FRAME2" library="frames" library_urn="urn:adsk.eagle:library:229" deviceset="FRAME_A_L" device=""/>
-<part name="R5" library="Ooo-Resistors" deviceset="RESISTOR_4PACK" device=""/>
+<part name="R5" library="Ooo-Resistors" deviceset="RESISTOR_4PACK" device="" value="10k"/>
 <part name="Q1" library="Ooo-Transistors" deviceset="MOSFET-N_DUAL" device=""/>
 <part name="U$18" library="Ooo-PowerSymbols" deviceset="3.3V" device=""/>
